File: Z80マイコン制作.kicad_pcb (KiCad board)
At the start: 2 copper layers, 150 x 150 mm, 87 parts, among them SW1 SW_DIP_x08, SW2 SW_DIP_x08, SW3 SW_DIP_x08, SW4 SW_Push, SW5 SW_Push, SW6 SW_DIP_x01, SW7 SW_DIP_x08, U1 Z80CPU, U11 74HCT244, U2 Z8420, U3 CY7C199, U4 74HCT244, U5 74HCT244, U6 74HCT244, U8 74LS06N, U9 74LS06N, Y1 CXO_DIP8

Commit message: 基盤確認済み、PCBに入りました
Parts:
- removed D10, D11, D12, D13, D14, D15, D16, D17, D18, D19, D20, D21, D22, D23, D24, D25, D26, D27, D28, D29, D30, D31, D8, D9: LED, LED_THT:LED_D3.0mm
- removed SW2, SW3: SW_DIP_x08, Package_DIP:CERDIP-16_W7.62mm_SideBrazed_Socket
- removed SW4, SW5: SW_Push, Button_Switch_THT:SW_PUSH_6mm
- removed SW6: SW_DIP_x01, Button_Switch_THT:SW_Slide-03_Wuerth-WS-SLTV_10x2.5x6.4_P2.54mm
- removed TP2: GND, TestPoint:TestPoint_THTPad_D2.0mm_Drill1.0mm
- removed Y1: CXO_DIP8, Oscillator:Oscillator_DIP-8
- added A0: LED, LED_THT:LED_D3.0mm, F.Cu at (114.8, 29.6)
- added A0-A7: SW_DIP_x08, Package_DIP:CERDIP-16_W7.62mm_SideBrazed_Socket, F.Cu at (-80.8, 44.1)
- added A1: LED, LED_THT:LED_D3.0mm, F.Cu at (110.4, 29.6)
- added A10: LED, LED_THT:LED_D3.0mm, F.Cu at (70.6, 29.6)
- added A11: LED, LED_THT:LED_D3.0mm, F.Cu at (66.2, 29.6)
- added A12: LED, LED_THT:LED_D3.0mm, F.Cu at (61.7, 29.6)
- added A13: LED, LED_THT:LED_D3.0mm, F.Cu at (57.3, 29.6)
- added A14: LED, LED_THT:LED_D3.0mm, F.Cu at (52.9, 29.6)
- added A2: LED, LED_THT:LED_D3.0mm, F.Cu at (105.9, 29.6)
- added A3: LED, LED_THT:LED_D3.0mm, F.Cu at (101.5, 29.6)
- added A4: LED, LED_THT:LED_D3.0mm, F.Cu at (97.1, 29.6)
- added A5: LED, LED_THT:LED_D3.0mm, F.Cu at (92.7, 29.6)
- added A6: LED, LED_THT:LED_D3.0mm, F.Cu at (88.3, 29.6)
- added A7: LED, LED_THT:LED_D3.0mm, F.Cu at (83.8, 29.6)
- added A8: LED, LED_THT:LED_D3.0mm, F.Cu at (79.4, 29.6)
- added A8-A14: SW_DIP_x08, Package_DIP:CERDIP-16_W7.62mm_SideBrazed_Socket, F.Cu at (-69.0, 44.1)
- added A9: LED, LED_THT:LED_D3.0mm, F.Cu at (75.0, 29.6)
- added BUSACK0: LED, LED_THT:LED_D3.0mm, F.Cu at (30.5, 124.5)
- added C0: 10uF, Capacitor_THT:CP_Radial_D5.0mm_P2.00mm, F.Cu at (36.3, 62.8)
- added C3: 0.01u, Capacitor_THT:CP_Radial_D5.0mm_P2.00mm, F.Cu at (-51.0, 121.6)
- added CLK0: LED, LED_THT:LED_D3.0mm, F.Cu at (30.5, 93.5)
- added D0: LED, LED_THT:LED_D3.0mm, F.Cu at (159.3, 76.9)
- added D0-D7: SW_DIP_x08, Package_DIP:CERDIP-16_W7.62mm_SideBrazed_Socket, F.Cu at (-57.3, 44.1)
- added I0-I7: SW_DIP_x08, Package_DIP:CERDIP-16_W7.62mm_SideBrazed_Socket, F.Cu at (-45.6, 44.1)
- added IORQ0: LED, LED_THT:LED_D3.0mm, F.Cu at (30.5, 120.0)
- added J0: Conn_01x08_Pin, Connector_PinHeader_2.54mm:PinHeader_1x08_P2.54mm_Vertical, F.Cu at (-44.4, 100.9)
- added J1: Conn_01x08_Pin, Connector_PinHeader_2.54mm:PinHeader_1x08_P2.54mm_Vertical, F.Cu at (-39.8, 100.9)
- added M0: LED, LED_THT:LED_D3.0mm, F.Cu at (30.5, 97.9)
- added MREQ0: LED, LED_THT:LED_D3.0mm, F.Cu at (30.5, 115.6)
- added O0: LED, LED_THT:LED_D3.0mm, F.Cu at (145.8, 77.0)
- added O1: LED, LED_THT:LED_D3.0mm, F.Cu at (145.8, 81.4)
- added O2: LED, LED_THT:LED_D3.0mm, F.Cu at (145.8, 85.8)
- added O3: LED, LED_THT:LED_D3.0mm, F.Cu at (145.8, 90.2)
- added O4: LED, LED_THT:LED_D3.0mm, F.Cu at (145.8, 94.6)
- added O5: LED, LED_THT:LED_D3.0mm, F.Cu at (145.8, 99.1)
- added O6: LED, LED_THT:LED_D3.0mm, F.Cu at (145.8, 103.5)
- added O7: LED, LED_THT:LED_D3.0mm, F.Cu at (145.8, 107.9)
- added R0: 4.7k, Resistor_THT:R_Axial_DIN0204_L3.6mm_D1.6mm_P7.62mm_Horizontal, F.Cu at (106.0, 34.3)
- added R31: 4.7k, Resistor_THT:R_Axial_DIN0204_L3.6mm_D1.6mm_P7.62mm_Horizontal, F.Cu at (-30.7, 93.9)
- added R32: 4.7k, Resistor_THT:R_Axial_DIN0204_L3.6mm_D1.6mm_P7.62mm_Horizontal, F.Cu at (-30.7, 97.1)
- added R33: 4.7k, Resistor_THT:R_Axial_DIN0204_L3.6mm_D1.6mm_P7.62mm_Horizontal, F.Cu at (-20.2, 65.6)
- added R34: 4.7k, Resistor_THT:R_Axial_DIN0204_L3.6mm_D1.6mm_P7.62mm_Horizontal, F.Cu at (-20.2, 68.7)
- added R35: 330, Resistor_THT:R_Axial_DIN0204_L3.6mm_D1.6mm_P7.62mm_Horizontal, F.Cu at (-20.2, 71.9)
- added R36: 4.7k, Resistor_THT:R_Axial_DIN0204_L3.6mm_D1.6mm_P7.62mm_Horizontal, F.Cu at (-20.2, 75.0)
- added R37: 4.7k, Resistor_THT:R_Axial_DIN0204_L3.6mm_D1.6mm_P7.62mm_Horizontal, F.Cu at (-20.2, 78.2)
- added R38: 4.7k, Resistor_THT:R_Axial_DIN0204_L3.6mm_D1.6mm_P7.62mm_Horizontal, F.Cu at (-20.2, 81.3)
- added R39: 10k, Resistor_THT:R_Axial_DIN0204_L3.6mm_D1.6mm_P7.62mm_Horizontal, F.Cu at (-20.2, 84.5)
- added R40: 4.7k, Resistor_THT:R_Axial_DIN0204_L3.6mm_D1.6mm_P7.62mm_Horizontal, F.Cu at (-6.64, 90.9)
- added RD0: LED, LED_THT:LED_D3.0mm, F.Cu at (30.5, 106.8)
- added RESET0: SW_Push, Button_Switch_THT:SW_PUSH_6mm, F.Cu at (29.8, 48.5)
- added RN0: 4.7k, Resistor_THT:R_Array_SIP9, F.Cu at (-119.4, 96.6)
- added RN6: 4.7k, Resistor_THT:R_Array_SIP9, F.Cu at (-119.4, 121.6)
- added RN7: 4.7k, Resistor_THT:R_Array_SIP9, F.Cu at (-119.4, 125.8)
- added RN8: 4.7k, Resistor_THT:R_Array_SIP9, F.Cu at (-119.4, 129.9)
- added RV0: R_Potentiometer, Potentiometer_THT:Potentiometer_ACP_CA9-H5_Horizontal, F.Cu at (29.2, 147.4)
- added TP0: VCC, TestPoint:TestPoint_THTPad_D2.0mm_Drill1.0mm, F.Cu at (43.2, 35.1)
- added U0: 74HCT244, Package_DIP:DIP-20_W7.62mm_Socket, F.Cu at (74.9, 53.3)
- added U10: 74HCT244, Package_DIP:DIP-20_W7.62mm_Socket, F.Cu at (-49.2, 17.0)
- added U13: NE555P, Package_DIP:DIP-8_W7.62mm, F.Cu at (40.6, 141.0)
- added U7: 74HCT244, Package_DIP:DIP-20_W7.62mm_Socket, F.Cu at (-17.8, 91.4)
- added WAIT0: LED, LED_THT:LED_D3.0mm, F.Cu at (30.5, 102.4)
- added WR0: LED, LED_THT:LED_D3.0mm, F.Cu at (30.5, 111.2)
- added WRITE0: SW_Push, Button_Switch_THT:SW_PUSH_6mm, F.Cu at (-35.5, 109.2)
- added Y0: CXO_DIP8, Oscillator:Oscillator_DIP-8, F.Cu at (41.9, 162.6)
- C1: value 10uF -> 100u
- C2: value 10u -> 0.01u
- R1, R2, R5: value R -> 4.7k
- R10, R11, R12, R13, R14, R15, R16, R17, R18, R19, R20, R21, R22, R23, R24, R25, R26, R27, R28, R29, R30, R8, R9: value 12k -> 4.7k
- R3, R4, R6, RN1, RN2, RN3, RN4, RN5: value 4.7ko -> 4.7k
- R7: value 330o -> 4.7k
- SW1: value SW_DIP_x08 -> SW_DIP_x01; footprint Package_DIP:CERDIP-16_W7.62mm_SideBrazed_Socket -> Button_Switch_THT:SW_Slide-03_Wuerth-WS-SLTV_10x2.5x6.4_P2.54mm
- SW7: value SW_DIP_x08 -> SW_Slide_DPDT; footprint Package_DIP:CERDIP-16_W7.62mm_SideBrazed_Socket -> Button_Switch_THT:SW_E-Switch_EG1271_SPDT
- TP1: value VCC -> GND
- U1: value Z80CPU -> 74HCT244; footprint Package_DIP:DIP-40_W15.24mm_Socket -> Package_DIP:DIP-20_W7.62mm_Socket
- U2: value Z8420 -> 74HCT244; footprint Package_DIP:DIP-40_W15.24mm_Socket -> Package_DIP:DIP-20_W7.62mm_Socket
- U3: value CY7C199 -> 74HCT244; footprint Package_DIP:DIP-28_W7.62mm_Socket -> Package_DIP:DIP-20_W7.62mm_Socket
- U4: value 74HCT244 -> Z80CPU; footprint Package_DIP:DIP-20_W7.62mm_Socket -> Package_DIP:DIP-40_W15.24mm_Socket
- U5: value 74HCT244 -> Z8420; footprint Package_DIP:DIP-20_W7.62mm_Socket -> Package_DIP:DIP-40_W15.24mm_Socket
- U6: value 74HCT244 -> CY7C199; footprint Package_DIP:DIP-20_W7.62mm_Socket -> Package_DIP:DIP-28_W7.62mm_Socket
- U8, U9: value 74LS06N -> 74HCT244; footprint Package_DIP:DIP-14_W7.62mm_Socket -> Package_DIP:DIP-20_W7.62mm_Socket
- moved RN1 259.7 mm to (-119.4, 100.7), turned to 0 degrees
- moved RN4 252.9 mm to (-119.4, 113.2), turned to 0 degrees
- moved RN2 250.7 mm to (-119.4, 104.9), turned to 0 degrees
- moved RN3 249.5 mm to (-119.4, 109.1), turned to 0 degrees
- moved RN5 221.3 mm to (-119.4, 117.4), turned to 0 degrees
- moved U2 201.0 mm to (-96.0, 17.0), turned to 0 degrees
- moved U9 186.9 mm to (-60.9, 17.0)
- moved U8 157.0 mm to (-75.9, 73.9)
- moved SW7 148.3 mm to (29.2, 170.0), turned to 90 degrees
- moved U11 139.3 mm to (-37.5, 17.0)
- moved C2 135.3 mm to (-51.0, 115.0)
- moved D7 128.0 mm to (159.3, 107.8)
- moved R15 123.2 mm to (-41.3, 78.2)
- moved R7 119.8 mm to (83.9, 34.3), turned to -90 degrees
- moved R5 114.1 mm to (90.2, 34.3), turned to -90 degrees
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Connections:
- C1 pad 1: Net-(U1-~{RESET}) -> VCC
- C2 pad 1: VCC -> Net-(U13-CV)
- C2 pad 2: GND -> Net-(U13-GND)
- D1 pad 1: Net-(D1-K) -> GND
- D2 pad 1: Net-(D2-K) -> GND
- D3 pad 1: Net-(D3-K) -> GND
- D4 pad 1: Net-(D4-K) -> GND
- D5 pad 1: Net-(D5-K) -> GND
- D6 pad 1: Net-(D6-K) -> GND
- R1 pad 1: VCC -> Net-(A1-A)
- R1 pad 2: Net-(U6-1Y0) -> Net-(U0-1Y1)
- R10 pad 2: Net-(U1-A2) -> Net-(U1-1Y2)
- R11 pad 2: Net-(U1-A3) -> Net-(U1-1Y3)
- R12 pad 2: Net-(U1-A4) -> Net-(U1-2Y0)
- R13 pad 2: Net-(U1-A5) -> Net-(U1-2Y1)
- R14 pad 2: Net-(U1-A6) -> Net-(U1-2Y2)
- R15 pad 2: Net-(U1-A7) -> Net-(U2-1Y0)
- R16 pad 1: Net-(D15-A) -> Net-(D1-A)
- R16 pad 2: Net-(U1-D0) -> Net-(U2-1Y1)
- R17 pad 1: Net-(D16-A) -> Net-(D2-A)
- R17 pad 2: Net-(U1-D1) -> Net-(U2-1Y2)
- R18 pad 1: Net-(D17-A) -> Net-(D3-A)
- R18 pad 2: Net-(U1-D2) -> Net-(U2-1Y3)
- R19 pad 1: Net-(D18-A) -> Net-(D4-A)
- R19 pad 2: Net-(U1-D3) -> Net-(U2-2Y0)
- R2 pad 1: VCC -> Net-(A2-A)
- R2 pad 2: Net-(U6-1Y1) -> Net-(U0-1Y2)
- R20 pad 1: Net-(D21-A) -> Net-(D5-A)
- R20 pad 2: Net-(U1-D4) -> Net-(U2-2Y1)
- R21 pad 1: Net-(D22-A) -> Net-(D6-A)
- R21 pad 2: Net-(U1-D5) -> Net-(U2-2Y2)
- R22 pad 1: Net-(D23-A) -> Net-(D7-A)
- R22 pad 2: Net-(U1-D6) -> Net-(U2-2Y3)
- R23 pad 2: Net-(U1-D7) -> Net-(U3-1Y0)
- R24 pad 2: Net-(U1-A14) -> Net-(U3-1Y1)
- R25 pad 2: Net-(U1-A13) -> Net-(U3-1Y2)
- R26 pad 2: Net-(U1-A12) -> Net-(U3-1Y3)
- R27 pad 2: Net-(U1-A11) -> Net-(U3-2Y0)
- R28 pad 2: Net-(U1-A10) -> Net-(U3-2Y1)
- R29 pad 2: Net-(U1-A9) -> Net-(U3-2Y2)
- R3 pad 1: VCC -> Net-(A3-A)
- R3 pad 2: Net-(U1-~{RESET}) -> Net-(U0-1Y3)
- R30 pad 2: Net-(U1-A8) -> Net-(U3-2Y3)
- R4 pad 1: VCC -> Net-(A4-A)
- R4 pad 2: Net-(U1-~{BUSRQ}) -> Net-(U0-2Y0)
- R5 pad 1: VCC -> Net-(A5-A)
- R5 pad 2: Net-(U1-~{NMI}) -> Net-(U0-2Y1)
- R6 pad 1: VCC -> Net-(A6-A)
- R6 pad 2: Net-(U2-IEI) -> Net-(U0-2Y2)
- R7 pad 1: Net-(U1-~{CLK}) -> Net-(A7-A)
- R7 pad 2: VCC -> Net-(U0-2Y3)
- R8 pad 1: Net-(D7-A) -> Net-(A8-A)
- R8 pad 2: Net-(U1-A0) -> Net-(U1-1Y0)
- R9 pad 2: Net-(U1-A1) -> Net-(U1-1Y1)
- RN2 pad 9: Net-(RN2-R8) -> unconnected-(RN2-R8-Pad9)
- RN3 pad 9: unconnected-(RN3-R8-Pad9) -> Net-(RN3-R8)
- RN4 pad 2: Net-(D1-A) -> Net-(RN4-R1)
- RN4 pad 3: Net-(D2-A) -> Net-(RN4-R2)
- RN4 pad 4: Net-(D3-A) -> Net-(RN4-R3)
- RN4 pad 5: Net-(D4-A) -> Net-(RN4-R4)
- RN4 pad 6: Net-(D5-A) -> Net-(RN4-R5)
- RN4 pad 7: Net-(D6-A) -> Net-(RN4-R6)
- RN4 pad 8: Net-(D19-A) -> Net-(RN4-R7)
- RN4 pad 9: Net-(D20-A) -> unconnected-(RN4-R8-Pad9)
- SW1 pad 1: Net-(RN5-R1) -> GND
- SW1 pad 2: Net-(RN5-R2) -> Net-(U4-~{BUSRQ})
- SW1 pad 3: Net-(RN5-R3) -> (no net)
- SW7 pad 1: Net-(RN3-R1) -> Net-(Y0-OUT)
- SW7 pad 2: Net-(RN3-R2) -> Net-(RN0-R1)
- SW7 pad 3: Net-(RN3-R3) -> Net-(U13-Q)
- SW7 pad 4: Net-(RN3-R4) -> Net-(U13-CV)
- SW7 pad 5: Net-(RN3-R5) -> GND
- SW7 pad 6: Net-(RN3-R6) -> Net-(Y0-GND)
- TP1 pad 1: VCC -> GND
- U1 pad 1: Net-(U1-A11) -> Net-(U0-1OE)
- U1 pad 10: Net-(U1-D6) -> GND
- U1 pad 11: VCC -> unconnected-(U1-2A3-Pad11)
- U1 pad 12: Net-(U1-D2) -> Net-(U1-1Y3)
- U1 pad 13: Net-(U1-D7) -> Net-(RN2-R7)
- U1 pad 14: Net-(U1-D0) -> Net-(U1-1Y2)
- U1 pad 15: Net-(U1-D1) -> Net-(RN2-R6)
- U1 pad 16: Net-(U1-~{INT}) -> Net-(U1-1Y1)
- U1 pad 17: Net-(U1-~{NMI}) -> Net-(RN2-R5)
- U1 pad 18: unconnected-(U1-~{HALT}-Pad18) -> Net-(U1-1Y0)
- U1 pad 19: Net-(U1-~{MREQ}) -> Net-(U0-1OE)
- U1 pad 2: Net-(U1-A12) -> Net-(RN2-R1)
- U1 pad 20: Net-(U1-~{IORQ}) -> VCC
- U1 pad 3: Net-(U1-A13) -> Net-(U1-2Y0)
- U1 pad 4: Net-(U1-A14) -> Net-(RN2-R2)
- U1 pad 5: unconnected-(U1-A15-Pad5) -> Net-(U1-2Y1)
- U1 pad 6: Net-(U1-~{CLK}) -> Net-(RN2-R3)
- U1 pad 7: Net-(U1-D4) -> Net-(U1-2Y2)
- U1 pad 8: Net-(U1-D3) -> Net-(RN2-R4)
- U1 pad 9: Net-(U1-D5) -> unconnected-(U1-2Y3-Pad9)
- U11 pad 1: Net-(U1-~{BUSACK}) -> Net-(RN0-R8)
- U11 pad 11: Net-(U1-A7) -> Net-(RN5-R8)
- U11 pad 12: Net-(RN1-R4) -> Net-(RN3-R4)
- U11 pad 13: Net-(U1-A6) -> Net-(RN5-R7)
- U11 pad 14: Net-(RN1-R3) -> Net-(RN3-R3)
- U11 pad 15: Net-(U1-A5) -> Net-(RN5-R6)
- U11 pad 16: Net-(RN1-R2) -> Net-(RN3-R2)
- U11 pad 17: Net-(U1-A4) -> Net-(RN5-R5)
- U11 pad 18: Net-(RN1-R1) -> Net-(RN3-R1)
- U11 pad 19: Net-(U1-~{BUSACK}) -> Net-(RN0-R8)
- U11 pad 2: Net-(U1-A0) -> Net-(RN5-R1)
- U11 pad 3: Net-(RN1-R5) -> Net-(RN3-R5)
- U11 pad 4: Net-(U1-A1) -> Net-(RN5-R2)
- U11 pad 5: Net-(RN1-R6) -> Net-(RN3-R6)
- U11 pad 6: Net-(U1-A2) -> Net-(RN5-R3)
- U11 pad 7: Net-(RN1-R7) -> Net-(RN3-R7)
- U11 pad 8: Net-(U1-A3) -> Net-(RN5-R4)
- U11 pad 9: Net-(RN1-R8) -> Net-(RN3-R8)
- U2 pad 1: Net-(U1-D2) -> Net-(U0-1OE)
- U2 pad 10: Net-(RN5-R5) -> GND
- U2 pad 11: GND -> Net-(RN1-R8)
- U2 pad 12: Net-(RN5-R4) -> Net-(U2-1Y3)
- U2 pad 13: Net-(RN5-R3) -> Net-(RN1-R7)
- U2 pad 14: Net-(RN5-R2) -> Net-(U2-1Y2)
- U2 pad 15: Net-(RN5-R1) -> Net-(RN1-R6)
- U2 pad 16: unconnected-(U2-~{ASTB}-Pad16) -> Net-(U2-1Y1)
- U2 pad 17: unconnected-(U2-~{BSTB}-Pad17) -> Net-(RN1-R5)
- U2 pad 18: unconnected-(U2-ARDY-Pad18) -> Net-(U2-1Y0)
- U2 pad 19: Net-(U1-D0) -> Net-(U0-1OE)
- U2 pad 2: Net-(U1-D7) -> Net-(RN1-R1)
- U2 pad 20: Net-(U1-D1) -> VCC
- U2 pad 3: Net-(U1-D6) -> Net-(U2-2Y0)
- U2 pad 4: Net-(U1-~{IORQ}) -> Net-(RN1-R2)
- U2 pad 5: Net-(U1-A1) -> Net-(U2-2Y1)
- U2 pad 6: Net-(U1-A0) -> Net-(RN1-R3)
- U2 pad 7: Net-(RN5-R8) -> Net-(U2-2Y2)
- U2 pad 8: Net-(RN5-R7) -> Net-(RN1-R4)
- U2 pad 9: Net-(RN5-R6) -> Net-(U2-2Y3)
- U3 pad 1: Net-(U1-A5) -> Net-(U0-1OE)
- U3 pad 10: Net-(U1-A14) -> GND
- U3 pad 11: Net-(U1-D0) -> Net-(RN0-R8)
- U3 pad 12: Net-(U1-D1) -> Net-(U3-1Y3)
- U3 pad 13: Net-(U1-D2) -> Net-(RN0-R7)
- U3 pad 14: GND -> Net-(U3-1Y2)
- U3 pad 15: Net-(U1-D3) -> Net-(RN0-R6)
- U3 pad 16: Net-(U1-D4) -> Net-(U3-1Y1)
- U3 pad 17: Net-(U1-D5) -> Net-(RN0-R5)
- U3 pad 18: Net-(U1-D6) -> Net-(U3-1Y0)
- U3 pad 19: Net-(U1-D7) -> Net-(U0-1OE)
- U3 pad 2: Net-(U1-A6) -> Net-(RN0-R1)
- U3 pad 20: Net-(U1-~{MREQ}) -> VCC
- U3 pad 3: Net-(U1-A7) -> Net-(U3-2Y0)
- U3 pad 4: Net-(U1-A8) -> Net-(RN0-R2)
- U3 pad 5: Net-(U1-A9) -> Net-(U3-2Y1)
- U3 pad 6: Net-(U1-A10) -> Net-(RN0-R3)
- U3 pad 7: Net-(U1-A11) -> Net-(U3-2Y2)
- U3 pad 8: Net-(U1-A12) -> Net-(RN0-R4)
- U3 pad 9: Net-(U1-A13) -> Net-(U3-2Y3)
- U4 pad 1: Net-(U1-~{BUSACK}) -> Net-(RN2-R4)
- U4 pad 10: GND -> Net-(RN1-R7)
- U4 pad 11: Net-(U1-D7) -> VCC
- U4 pad 12: Net-(RN2-R4) -> Net-(RN1-R3)
- U4 pad 13: Net-(U1-D6) -> Net-(RN1-R8)
- U4 pad 14: Net-(RN2-R3) -> Net-(RN1-R1)
- U4 pad 15: Net-(U1-D5) -> Net-(RN1-R2)
- U4 pad 16: Net-(RN2-R2) -> Net-(U4-~{INT})
- U4 pad 17: Net-(U1-D4) -> Net-(RN0-R3)
- U4 pad 18: Net-(RN2-R1) -> unconnected-(U4-~{HALT}-Pad18)
- U4 pad 19: Net-(U1-~{BUSACK}) -> Net-(RN0-R6)
- U4 pad 2: Net-(U1-D0) -> Net-(RN2-R5)
- U4 pad 20: VCC -> Net-(RN0-R7)
- U4 pad 3: Net-(RN2-R5) -> Net-(RN2-R6)
- U4 pad 4: Net-(U1-D1) -> Net-(RN2-R7)
- U4 pad 5: Net-(RN2-R6) -> unconnected-(U4-A15-Pad5)
- U4 pad 6: Net-(U1-D2) -> Net-(RN0-R1)
- U4 pad 7: Net-(RN2-R7) -> Net-(RN1-R5)
- U4 pad 8: Net-(U1-D3) -> Net-(RN1-R4)
- U4 pad 9: Net-(RN2-R8) -> Net-(RN1-R6)
- U5 pad 1: Net-(U1-~{BUSACK}) -> Net-(RN1-R3)
- U5 pad 10: GND -> Net-(J1-Pin_4)
- U5 pad 11: unconnected-(U5-2A3-Pad11) -> GND
- U5 pad 12: Net-(RN3-R4) -> Net-(J1-Pin_5)
- U5 pad 13: Net-(U1-A14) -> Net-(J1-Pin_6)
- U5 pad 14: Net-(RN3-R3) -> Net-(J1-Pin_7)
- U5 pad 15: Net-(U1-A13) -> Net-(J1-Pin_8)
- U5 pad 16: Net-(RN3-R2) -> unconnected-(U5-~{ASTB}-Pad16)
- U5 pad 17: Net-(U1-A12) -> unconnected-(U5-~{BSTB}-Pad17)
- U5 pad 18: Net-(RN3-R1) -> unconnected-(U5-ARDY-Pad18)
- U5 pad 19: Net-(U1-~{BUSACK}) -> Net-(RN1-R1)
- U5 pad 2: Net-(U1-A8) -> Net-(RN1-R8)
- U5 pad 20: VCC -> Net-(RN1-R2)
- U5 pad 3: Net-(RN3-R5) -> Net-(RN1-R7)
- U5 pad 4: Net-(U1-A9) -> Net-(RN0-R7)
- U5 pad 5: Net-(RN3-R6) -> Net-(RN3-R2)
- U5 pad 6: Net-(U1-A10) -> Net-(RN3-R1)
- U5 pad 7: Net-(RN3-R7) -> Net-(J1-Pin_1)
- U5 pad 8: Net-(U1-A11) -> Net-(J1-Pin_2)
- U5 pad 9: unconnected-(U5-2Y3-Pad9) -> Net-(J1-Pin_3)
- U6 pad 1: Net-(U1-~{BUSACK}) -> Net-(RN3-R6)
- U6 pad 10: GND -> Net-(RN2-R7)
- U6 pad 11: unconnected-(U6-2A3-Pad11) -> Net-(RN1-R1)
- U6 pad 12: unconnected-(U6-1Y3-Pad12) -> Net-(RN1-R2)
- U6 pad 13: unconnected-(U6-2A2-Pad13) -> Net-(RN1-R3)
- U6 pad 15: unconnected-(U6-2A1-Pad15) -> Net-(RN1-R4)
- U6 pad 16: Net-(U6-1Y1) -> Net-(RN1-R5)
- U6 pad 17: unconnected-(U6-2A0-Pad17) -> Net-(RN1-R6)
- U6 pad 18: Net-(U6-1Y0) -> Net-(RN1-R7)
- U6 pad 19: Net-(U1-~{BUSACK}) -> Net-(RN1-R8)
- U6 pad 2: Net-(U1-~{RD}) -> Net-(RN3-R7)
- U6 pad 20: VCC -> Net-(RN0-R6)
- U6 pad 3: unconnected-(U6-2Y0-Pad3) -> Net-(RN3-R8)
- U6 pad 4: Net-(U1-~{WR}) -> Net-(RN2-R1)
- U6 pad 5: unconnected-(U6-2Y1-Pad5) -> Net-(RN2-R2)
- U6 pad 6: Net-(U1-~{MREQ}) -> Net-(RN2-R3)
- U6 pad 7: unconnected-(U6-2Y2-Pad7) -> Net-(RN2-R4)
- U6 pad 8: unconnected-(U6-1A3-Pad8) -> Net-(RN2-R5)
- U6 pad 9: unconnected-(U6-2Y3-Pad9) -> Net-(RN2-R6)
- U8 pad 1: Net-(U2-PB0) -> Net-(RN0-R8)
- U8 pad 10: Net-(D5-K) -> GND
- U8 pad 11: Net-(U2-PB4) -> Net-(RN8-R1)
- U8 pad 12: Net-(D6-K) -> Net-(RN1-R4)
- U8 pad 13: Net-(U2-PB5) -> Net-(RN8-R2)
- U8 pad 14: VCC -> Net-(RN1-R3)
- U8 pad 2: Net-(D1-K) -> Net-(RN8-R8)
- U8 pad 3: Net-(U2-PB1) -> Net-(RN1-R5)
- U8 pad 4: Net-(D2-K) -> Net-(RN8-R7)
- U8 pad 5: Net-(U2-PB2) -> Net-(RN1-R6)
- U8 pad 6: Net-(D3-K) -> Net-(RN8-R6)
- U8 pad 7: GND -> Net-(RN1-R7)
- U8 pad 8: Net-(D4-K) -> Net-(RN8-R5)
- U8 pad 9: Net-(U2-PB3) -> Net-(RN1-R8)
- U9 pad 1: Net-(U2-PB6) -> Net-(RN0-R8)
- U9 pad 10: unconnected-(U9-Pad10) -> GND
- U9 pad 12: unconnected-(U9-Pad12) -> Net-(RN2-R4)
- U9 pad 13: unconnected-(U9-Pad13) -> Net-(RN4-R7)
- U9 pad 14: VCC -> Net-(RN2-R3)
- U9 pad 2: Net-(D19-K) -> Net-(RN4-R1)
- U9 pad 3: Net-(U2-PB7) -> Net-(RN2-R5)
- U9 pad 4: Net-(D20-K) -> Net-(RN4-R2)
- U9 pad 5: unconnected-(U9-Pad5) -> Net-(RN2-R6)
- U9 pad 6: unconnected-(U9-Pad6) -> Net-(RN4-R3)
- U9 pad 7: GND -> Net-(RN2-R7)
- U9 pad 8: unconnected-(U9-Pad8) -> Net-(RN4-R4)
Routing:
- net GND: track 688.3 -> 0.00 mm, vias 4 -> 0
- net VCC: track 563.7 -> 0.00 mm, vias 3 -> 0
- net Net-(U1-D2): track 205.3 -> 0.00 mm, vias 3 -> 0
- net Net-(U1-A0): track 184.1 -> 0.00 mm, vias 2 -> 0
- net Net-(U1-D3): track 181.8 -> 0.00 mm, vias 2 -> 0
- net Net-(U1-D7): track 179.8 -> 0.00 mm, vias 1 -> 0
- net Net-(U1-A1): track 177.6 -> 0.00 mm, vias 2 -> 0
- net Net-(U1-D4): track 174.8 -> 0.00 mm
- net Net-(U1-~{BUSACK}): track 173.8 -> 0.00 mm
- net Net-(U1-D6): track 171.1 -> 0.00 mm, vias 2 -> 0
- net Net-(U1-D5): track 167.3 -> 0.00 mm
- net Net-(U1-D0): track 166.2 -> 0.00 mm, vias 1 -> 0
- net Net-(U1-~{RD}): track 142.9 -> 0.00 mm, vias 1 -> 0
- net Net-(U1-D1): track 142.3 -> 0.00 mm, vias 1 -> 0
- net Net-(U1-A12): track 140.5 -> 0.00 mm, vias 4 -> 0
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
Commit message: ちょっと変えた
Parts:
- moved A0-A7 242.1 mm to (161.3, 49.5)
- moved D0-D7 234.7 mm to (161.8, 128.3)
- moved A8-A14 234.1 mm to (162.1, 81.5)
- moved U8 223.1 mm to (141.0, 126.2)
- moved U2 217.5 mm to (118.6, 51.9)
- moved U9 214.4 mm to (140.8, 89.7)
- moved R15 205.1 mm to (159.1, 34.5), turned to -90 degrees
- moved R16 202.7 mm to (156.0, 34.5), turned to -90 degrees
- moved I0-I7 200.5 mm to (108.5, 172.5), turned to 90 degrees
- moved R17 200.4 mm to (152.8, 34.5), turned to -90 degrees
- moved R18 198.2 mm to (149.7, 34.5), turned to -90 degrees
- moved WRITE0 197.9 mm to (162.4, 110.7)
- moved R19 196.0 mm to (146.5, 34.5), turned to -90 degrees
- moved J0 195.6 mm to (141.7, 161.0), turned to 90 degrees
- moved R20 194.0 mm to (143.4, 34.5), turned to -90 degrees
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
Commit message: 基盤のVCC,GND配線終わりました
Parts:
- removed J0, J1: Conn_01x08_Pin, Connector_PinHeader_2.54mm:PinHeader_1x08_P2.54mm_Vertical
- added PA: Conn_01x10_Pin, Connector_PinHeader_2.54mm:PinHeader_1x10_P2.54mm_Vertical, F.Cu at (131.3, 172.6)
- added PB: Conn_01x10_Pin, Connector_PinHeader_2.54mm:PinHeader_1x10_P2.54mm_Vertical, F.Cu at (173.4, 172.6)
- A14-A8: renamed from A8-A14; footprint Package_DIP:CERDIP-16_W7.62mm_SideBrazed_Socket -> Package_DIP:DIP-16_W7.62mm_Socket
- A7-A0: renamed from A0-A7; footprint Package_DIP:CERDIP-16_W7.62mm_SideBrazed_Socket -> Package_DIP:DIP-16_W7.62mm_Socket
- Crystal Oscillator: renamed from Y0
- D7-D0: renamed from D0-D7; footprint Package_DIP:CERDIP-16_W7.62mm_SideBrazed_Socket -> Package_DIP:DIP-16_W7.62mm_Socket
- I7-I0: renamed from I0-I7; footprint Package_DIP:CERDIP-16_W7.62mm_SideBrazed_Socket -> Package_DIP:DIP-16_W7.62mm_Socket
- NE555P: renamed from U13; footprint Package_DIP:DIP-8_W7.62mm -> Package_DIP:DIP-8_W7.62mm_Socket
- moved RN6 289.3 mm to (168.8, 147.2), turned to -90 degrees
- moved RN5 283.4 mm to (155.9, 49.9), turned to -90 degrees
- moved RN4 277.4 mm to (155.9, 79.0), turned to -90 degrees
- moved RN8 277.4 mm to (157.5, 146.6), turned to 90 degrees
- moved RN7 256.2 mm to (135.9, 147.2), turned to -90 degrees
- moved RN1 231.4 mm to (111.3, 81.5)
- moved RN3 194.5 mm to (73.4, 83.2)
- moved RN2 175.5 mm to (54.4, 80.0)
- moved RN0 155.3 mm to (35.3, 83.2)
- moved R37 122.0 mm to (62.7, 167.7)
- moved R35 121.1 mm to (70.4, 152.4), turned to 180 degrees
- moved R39 120.3 mm to (62.7, 171.6)
- moved R36 118.8 mm to (62.7, 160.1)
- moved R32 114.9 mm to (62.7, 163.9)
- moved R34 112.4 mm to (62.7, 144.7)
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- renumbered C2 to 0.01uF, C3 to 0.01uF, C1 to 100uF, C0 to 10uF, U10 to 74HCT244, U1 to 74HCT244, U3 to 74HCT244, U2 to 74HCT244, U11 to 74HCT244, U9 to 74HCT244, U0 to 74HCT244, U8 to 74HCT244, U7 to 74HCT244, BUSACK0 to BUSACK, SW1 to BUSRQ, CLK0 to CLK, SW7 to CLOCK_ch, U6 to CY7C199, RV0 to FREQUENCY, TP1 to GND, IORQ0 to IORQ, M0 to M1, MREQ0 to MREQ, RD0 to RD, RESET0 to RESET, TP0 to VCC, WAIT0 to WAIT, WR0 to WR, WRITE0 to WRITE, U4 to Z80CPU, U5 to Z80PIO
Connections:
- 74HCT244 pad 10: unconnected-(U7-GND-Pad10) -> GND
- 74HCT244 pad 20: unconnected-(U7-VCC-Pad20) -> VCC
Routing:
- net GND: track 0.00 -> 827.0 mm, vias 0 -> 1
- net VCC: track 0.00 -> 642.4 mm, vias 0 -> 2
Other:
- board text added: "NE555"
- board text added: "OFF"
- board text added: "ON"
- board text added: "OSC"

Commit message: ちょっと変更
Parts:
- renumbered 0.01uF to 0.01uF-0, 0.01uF to 0.01uF-1, 74HCT244 to 74HCT244-0, 74HCT244 to 74HCT244-1, 74HCT244 to 74HCT244-2, 74HCT244 to 74HCT244-3, 74HCT244 to 74HCT244-4, 74HCT244 to 74HCT244-5, 74HCT244 to 74HCT244-6, 74HCT244 to 74HCT244-7, 74HCT244 to 74HCT244-8
Changed lines of the file:
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@@
 		(descr "CP, Radial series, Radial, pin pitch=2.00mm, diameter=5mm, height=7mm, Electrolytic Capacitor")
 		(tags "CP Radial series Radial pin pitch 2.00mm diameter 5mm height 7mm Electrolytic Capacitor")
-		(property "Reference" "0.01uF"
+		(property "Reference" "0.01uF-1"
 			(at 1 -3.75 0)
 			(layer "F.SilkS")
@@
 		(descr "20-lead though-hole mounted DIP package, row spacing 7.62mm (300 mils), Socket")
 		(tags "THT DIP DIL PDIP 2.54mm 7.62mm 300mil Socket")
-		(property "Reference" "74HCT244"
+		(property "Reference" "74HCT244-5"
 			(at 3.81 -2.33 0)
 			(layer "F.SilkS")
@@
 		(descr "20-lead though-hole mounted DIP package, row spacing 7.62mm (300 mils), Socket")
 		(tags "THT DIP DIL PDIP 2.54mm 7.62mm 300mil Socket")
-		(property "Reference" "74HCT244"
+		(property "Reference" "74HCT244-1"
 			(at 3.81 -2.33 0)
 			(layer "F.SilkS")
@@
 		(descr "20-lead though-hole mounted DIP package, row spacing 7.62mm (300 mils), Socket")
 		(tags "THT DIP DIL PDIP 2.54mm 7.62mm 300mil Socket")
-		(property "Reference" "74HCT244"
+		(property "Reference" "74HCT244-0"
 			(at 3.81 -2.33 0)
 			(layer "F.SilkS")
@@
 		(descr "20-lead though-hole mounted DIP package, row spacing 7.62mm (300 mils), Socket")
 		(tags "THT DIP DIL PDIP 2.54mm 7.62mm 300mil Socket")
-		(property "Reference" "74HCT244"
+		(property "Reference" "74HCT244-3"
 			(at 3.81 -2.33 0)
 			(layer "F.SilkS")
@@
 		(descr "20-lead though-hole mounted DIP package, row spacing 7.62mm (300 mils), Socket")
 		(tags "THT DIP DIL PDIP 2.54mm 7.62mm 300mil Socket")
-		(property "Reference" "74HCT244"
+		(property "Reference" "74HCT244-4"
 			(at 3.81 -2.33 0)
 			(layer "F.SilkS")
@@
 		(descr "CP, Radial series, Radial, pin pitch=2.00mm, diameter=5mm, height=7mm, Electrolytic Capacitor")
 		(tags "CP Radial series Radial pin pitch 2.00mm diameter 5mm height 7mm Electrolytic Capacitor")
-		(property "Reference" "0.01uF"
+		(property "Reference" "0.01uF-0"
 			(at 1 -3.75 0)
 			(layer "F.SilkS")
@@
 		(descr "20-lead though-hole mounted DIP package, row spacing 7.62mm (300 mils), Socket")
 		(tags "THT DIP DIL PDIP 2.54mm 7.62mm 300mil Socket")
-		(property "Reference" "74HCT244"
+		(property "Reference" "74HCT244-6"
 			(at 3.81 -2.33 0)
 			(layer "F.SilkS")
@@
 		(descr "20-lead though-hole mounted DIP package, row spacing 7.62mm (300 mils), Socket")
 		(tags "THT DIP DIL PDIP 2.54mm 7.62mm 300mil Socket")
-		(property "Reference" "74HCT244"
+		(property "Reference" "74HCT244-2"
 			(at 3.81 -2.33 0)
 			(layer "F.SilkS")
@@
 		(descr "20-lead though-hole mounted DIP package, row spacing 7.62mm (300 mils), Socket")
 		(tags "THT DIP DIL PDIP 2.54mm 7.62mm 300mil Socket")
-		(property "Reference" "74HCT244"
+		(property "Reference" "74HCT244-8"
 			(at 3.81 -2.33 0)
 			(layer "F.SilkS")
@@
 		(descr "20-lead though-hole mounted DIP package, row spacing 7.62mm (300 mils), Socket")
 		(tags "THT DIP DIL PDIP 2.54mm 7.62mm 300mil Socket")
-		(property "Reference" "74HCT244"
+		(property "Reference" "74HCT244-7"
 			(at 3.81 -2.33 0)
 			(layer "F.SilkS")

Commit message: 基盤完成
Parts:
- moved R30 1.27 mm to (38.7, 121.2)
- moved R22 1.09 mm to (142.0, 34.3)
- moved R23 1.06 mm to (38.7, 96.8)
- moved R15 0.96 mm to (166.0, 34.3)
- moved R29 0.94 mm to (38.7, 117.7)
- moved R24 0.73 mm to (38.7, 100.3)
- moved R21 0.71 mm to (145.4, 34.3)
- moved R16 0.68 mm to (162.6, 34.3)
- moved R28 0.60 mm to (38.7, 114.2)
- moved R20 0.44 mm to (148.8, 34.3)
- moved R17 0.40 mm to (159.1, 34.3)
- moved R25 0.40 mm to (38.7, 103.7)
- moved R27 0.27 mm to (38.7, 110.7)
- moved R19 0.16 mm to (152.3, 34.3)
- moved R18 0.12 mm to (155.7, 34.3)
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Routing:
- net Net-(RN1-R1): track 0.00 -> 266.2 mm, vias 0 -> 3
- net Net-(RN0-R8): track 0.00 -> 260.9 mm, vias 0 -> 5
- net Net-(RN1-R2): track 0.00 -> 257.6 mm, vias 0 -> 4
- net Net-(RN1-R6): track 0.00 -> 210.7 mm, vias 0 -> 3
- net Net-(U0-1OE): track 0.00 -> 210.3 mm, vias 0 -> 2
- net Net-(RN0-R4): track 0.00 -> 206.5 mm, vias 0 -> 1
- net Net-(RN1-R7): track 0.00 -> 202.3 mm, vias 0 -> 3
- net Net-(RN0-R5): track 0.00 -> 202.2 mm, vias 0 -> 4
- net Net-(RN1-R4): track 0.00 -> 193.5 mm, vias 0 -> 2
- net Net-(RN0-R1): track 0.00 -> 192.1 mm, vias 0 -> 1
- net Net-(RN0-R6): track 0.00 -> 189.6 mm, vias 0 -> 5
- net Net-(RN1-R3): track 0.00 -> 187.5 mm, vias 0 -> 2
- net Net-(RN1-R5): track 0.00 -> 183.2 mm, vias 0 -> 2
- net Net-(RN3-R1): track 0.00 -> 181.2 mm, vias 0 -> 2
- net Net-(RN1-R8): track 0.00 -> 180.7 mm, vias 0 -> 2
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
Commit message: 今度こそ基盤完成！！
Parts:
- removed RN6: 4.7k, Resistor_THT:R_Array_SIP9
- added R41: 4.7k, Resistor_THT:R_Axial_DIN0204_L3.6mm_D1.6mm_P7.62mm_Horizontal, F.Cu at (163.7, 168.3)
- added R42: 4.7k, Resistor_THT:R_Axial_DIN0204_L3.6mm_D1.6mm_P7.62mm_Horizontal, F.Cu at (160.6, 168.3)
- added R43: 4.7k, Resistor_THT:R_Axial_DIN0204_L3.6mm_D1.6mm_P7.62mm_Horizontal, F.Cu at (157.4, 168.3)
- added R44: 4.7k, Resistor_THT:R_Axial_DIN0204_L3.6mm_D1.6mm_P7.62mm_Horizontal, F.Cu at (154.2, 168.3)
- added R45: 4.7k, Resistor_THT:R_Axial_DIN0204_L3.6mm_D1.6mm_P7.62mm_Horizontal, F.Cu at (151.1, 168.3)
- added R46: 4.7k, Resistor_THT:R_Axial_DIN0204_L3.6mm_D1.6mm_P7.62mm_Horizontal, F.Cu at (147.9, 168.3)
- added R47: 4.7k, Resistor_THT:R_Axial_DIN0204_L3.6mm_D1.6mm_P7.62mm_Horizontal, F.Cu at (144.8, 168.3)
- added R48: 4.7k, Resistor_THT:R_Axial_DIN0204_L3.6mm_D1.6mm_P7.62mm_Horizontal, F.Cu at (141.7, 168.3)
- CLOCK ch: renamed from CLOCK_ch
- OSCILLATOR: renamed from Crystal Oscillator
- Z80 CPU: renamed from Z80CPU
- moved O7 31.0 mm to (168.1, 173.0)
- moved O0 30.9 mm to (137.2, 173.0)
- moved O6 22.2 mm to (163.7, 173.0)
- moved O1 22.0 mm to (141.6, 173.0)
- moved O5 13.3 mm to (159.3, 173.0)
- moved O2 13.2 mm to (146.0, 173.0)
- moved O4 4.49 mm to (154.9, 173.0)
- moved O3 4.35 mm to (150.5, 173.0)
- renumbered 0.01uF-1 to 0.01uF, 0.01uF-0 to 0.01uF, FREQUENCY to FREQENCY, NE555P to UNE555P
Connections:
- 74HCT244-7 pad 12: Net-(J1-Pin_7) -> Net-(74HCT244-7-1Y3)
- 74HCT244-7 pad 14: Net-(J1-Pin_8) -> Net-(74HCT244-7-1Y2)
- 74HCT244-7 pad 16: Net-(J1-Pin_9) -> Net-(74HCT244-7-1Y1)
- 74HCT244-7 pad 18: Net-(J1-Pin_10) -> Net-(74HCT244-7-1Y0)
- 74HCT244-7 pad 3: Net-(J1-Pin_6) -> Net-(74HCT244-7-2Y0)
- 74HCT244-7 pad 5: Net-(J1-Pin_5) -> Net-(74HCT244-7-2Y1)
- 74HCT244-7 pad 7: Net-(J1-Pin_4) -> Net-(74HCT244-7-2Y2)
- 74HCT244-7 pad 9: Net-(J1-Pin_3) -> Net-(74HCT244-7-2Y3)
- O0 pad 2: Net-(J1-Pin_3) -> Net-(O0-A)
- O1 pad 2: Net-(J1-Pin_4) -> Net-(O1-A)
- O2 pad 2: Net-(J1-Pin_5) -> Net-(O2-A)
- O3 pad 2: Net-(J1-Pin_6) -> Net-(O3-A)
- O4 pad 2: Net-(J1-Pin_7) -> Net-(O4-A)
- O5 pad 2: Net-(J1-Pin_8) -> Net-(O5-A)
- O6 pad 2: Net-(J1-Pin_9) -> Net-(O6-A)
- O7 pad 2: Net-(J1-Pin_10) -> Net-(O7-A)
- PB pad 10: Net-(J1-Pin_10) -> Net-(74HCT244-7-1Y0)
- PB pad 3: Net-(J1-Pin_3) -> Net-(74HCT244-7-2Y3)
- PB pad 4: Net-(J1-Pin_4) -> Net-(74HCT244-7-2Y2)
- PB pad 5: Net-(J1-Pin_5) -> Net-(74HCT244-7-2Y1)
- PB pad 6: Net-(J1-Pin_6) -> Net-(74HCT244-7-2Y0)
- PB pad 7: Net-(J1-Pin_7) -> Net-(74HCT244-7-1Y3)
- PB pad 8: Net-(J1-Pin_8) -> Net-(74HCT244-7-1Y2)
- PB pad 9: Net-(J1-Pin_9) -> Net-(74HCT244-7-1Y1)
Routing:
- net Net-(J1-Pin_6): track 98.7 -> 0.00 mm, vias 2 -> 0
- net Net-(J1-Pin_9): track 91.0 -> 0.00 mm, vias 1 -> 0
- net Net-(74HCT244-7-2Y0): track 0.00 -> 87.4 mm, vias 0 -> 1
- net Net-(J1-Pin_5): track 84.5 -> 0.00 mm, vias 2 -> 0
- net Net-(J1-Pin_10): track 79.4 -> 0.00 mm, vias 1 -> 0
- net Net-(J1-Pin_8): track 78.4 -> 0.00 mm, vias 2 -> 0
- net Net-(J1-Pin_4): track 76.2 -> 0.00 mm, vias 2 -> 0
- net Net-(J1-Pin_3): track 72.3 -> 0.00 mm, vias 1 -> 0
- net Net-(74HCT244-7-1Y0): track 0.00 -> 71.1 mm
- net Net-(J1-Pin_7): track 70.7 -> 0.00 mm, vias 1 -> 0
- net Net-(74HCT244-7-2Y1): track 0.00 -> 70.4 mm, vias 0 -> 2
- net Net-(74HCT244-7-2Y3): track 0.00 -> 70.3 mm, vias 0 -> 1
- net Net-(74HCT244-7-2Y2): track 0.00 -> 69.0 mm, vias 0 -> 3
- net Net-(74HCT244-7-1Y1): track 0.00 -> 65.5 mm, vias 0 -> 1
- net Net-(74HCT244-7-1Y2): track 0.00 -> 61.4 mm, vias 0 -> 1
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Other:
- board text added: "GND"
- board text added: "I0"
- board text added: "I1"
- board text added: "I2"
- board text added: "I3"
- board text added: "I4"
- board text added: "I5"
- board text added: "I6"
- board text added: "I7"
- board text added: "O0"
- board text added: "O1"
- board text added: "O2"
- board text added: "O3"
- board text added: "O4"
- board text added: "O5"
- board text added: "O6"
- board text added: "O7"
- board text added: "VCC"
