File: Z80マイコン制作.kicad_pcb (KiCad board)
At the start: 2 copper layers, 150 x 150 mm, 127 parts, among them M1 LED

Commit message: start designing
Parts:
- moved Z80PIO 139.8 mm to (221.0, 81.3)
- moved Z80 CPU 128.5 mm to (182.9, 94.0)
- moved A1 127.3 mm to (236.4, 47.4)
- moved A10 127.3 mm to (196.6, 47.4)
- moved A11 127.3 mm to (192.2, 47.4)
- moved A13 127.3 mm to (183.4, 47.4)
- moved A4 127.3 mm to (223.1, 47.4)
- moved A6 127.3 mm to (214.3, 47.4)
- moved A8 127.3 mm to (205.5, 47.4)
- moved R12 127.3 mm to (194.3, 52.1)
- moved R13 127.3 mm to (191.1, 52.1)
- moved R2 127.3 mm to (225.7, 52.1)
- moved R3 127.3 mm to (222.6, 52.1)
- moved R7 127.3 mm to (210.0, 52.1)
- moved R8 127.3 mm to (206.8, 52.1)
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Routing:
- net GND: track 944.5 -> 0.00 mm, vias 1 -> 0
- net VCC: track 660.8 -> 0.00 mm, vias 3 -> 0
- net Net-(RN1-R1): track 266.2 -> 0.00 mm, vias 3 -> 0
- net Net-(RN0-R8): track 260.9 -> 0.00 mm, vias 5 -> 0
- net Net-(RN1-R2): track 257.6 -> 0.00 mm, vias 4 -> 0
- net Net-(RN1-R6): track 210.7 -> 0.00 mm, vias 3 -> 0
- net Net-(U0-1OE): track 210.3 -> 0.00 mm, vias 2 -> 0
- net Net-(RN0-R4): track 206.5 -> 0.00 mm, vias 1 -> 0
- net Net-(RN1-R7): track 202.3 -> 0.00 mm, vias 3 -> 0
- net Net-(RN0-R5): track 202.2 -> 0.00 mm, vias 4 -> 0
- net Net-(RN1-R4): track 193.5 -> 0.00 mm, vias 2 -> 0
- net Net-(RN0-R1): track 192.4 -> 0.00 mm, vias 1 -> 0
- net Net-(RN0-R6): track 189.6 -> 0.00 mm, vias 5 -> 0
- net Net-(RN1-R3): track 187.5 -> 0.00 mm, vias 2 -> 0
- net Net-(RN1-R5): track 183.2 -> 0.00 mm, vias 2 -> 0
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Other:
- board size 150 x 150 mm -> 100 x 100 mm
- board text removed: "GND"
- board text removed: "I0"
- board text removed: "I1"
- board text removed: "I2"
- board text removed: "I3"
- board text removed: "I4"
- board text removed: "I5"
- board text removed: "I6"
- board text removed: "I7"
- board text removed: "NE555"
- board text removed: "O0"
- board text removed: "O1"
- board text removed: "O2"
- board text removed: "O3"
- board text removed: "O4"
- board text removed: "O5"
- board text removed: "O6"
- board text removed: "O7"
- board text removed: "OFF"
- board text removed: "ON"
- board text removed: "OSC"
- board text removed: "VCC"
- board text removed: "電子技術研究部 Z80マイコン制作"
